File: smart-home.matherboard.brd (EAGLE design)
At the start: 78 x 54 mm, 6 parts

Commit message: Prepea
Parts:
- removed R1: 10kOm, rcl:R0603
- removed U$3: E18-MS1PA1IPX, e18-ms1pa1-ipx:E18-MS1PA1-IPX
- added C101, C211, C241, C271, C311: C_100N_0402_X5R_K_10, rcl:C0402
- added C201: C_1N_0402_NP0_J_50, rcl:C0402
- added C21, C31: C_47P_0402_NP0_J_50, rcl:C0402
- added C221, C231: C_27P_0402_NP0_J_50, rcl:C0402
- added C272: C_220P_0402_NP0_J_50, rcl:C0402
- added C391, C401: C_1U_0402_X5R_K_6P3, rcl:C0402
- added C4: C_2U2_0402_X5R_M_4VDC, rcl:C0402
- added C41: C_10P_0402_NP0_J_50, rcl:C0402
- added C5: C_0P5_0402_NP0_B_50, rcl:C0402
- added IC1: CC2531, texas:RHA_S-PVQFN-N40
- added L1: L_BEAD_102_0402, rcl:L0402
- added L301: L_6N8_0402_J, rcl:L0402
- added R201: R_2K2_0402_G, rcl:R0402
- added R21, R31: R_33_0402_G, rcl:R0402
- added R301: R_56K_0402_F, rcl:R0402
- added R32: R_1K5_0402_G, rcl:R0402
- added R9: R_0_0402, rcl:R0402
- added U$4: MEANDER-ANT, Antennas:MEANDER-ANT
- added U1: JTI_2450BM15A0002, texas_instruments:JTI_2450BM15A0002
- added USB1: MOLEX-47364-0001, Конекторы:MOLEX-47364-0001
- added X1: NX3225SA, Crystals:NX32256A
Connections:
- removed net CSN: U$3.P1.4
- removed net DC: U$1.36, U$3.P2.2
- removed net DD: U$1.38, U$3.P2.1
- removed net E18-RX: U$1.8, U$3.P0.2
- removed net E18-TX: U$1.10, U$3.P0.3
- removed net MISO: U$3.P1.7
- removed net MOSI: U$3.P1.6
- removed net RST: R1.1, U$1.35, U$3.RST
- removed net SCK: U$3.P1.5
- new net CC_DN: R21.1, USB1.2
- new net CC_DP: R31.1, USB1.3
- new net N$10: L301.2, R301.2
- new net N$11: IC1.25, U1.P$4
- new net N$12: IC1.26, U1.P$3
- new net N$13: C5.1, R9.1, U1.P$1
- new net N$14: R9.2, U$4.FEED
- new net N$15: C101.1, C211.1, C241.1, C271.1, C272.1, C311.1, C391.1, C4.1, C41.1, IC1.10, IC1.21, IC1.24, IC1.27, IC1.28, IC1.29, IC1.31, IC1.39, IC1.4, L1.2
- new net N$16: USB1.1
- new net N$3: C31.1, IC1.2, R31.2, R32.2
- new net N$4: C21.1, IC1.3, R21.2
- new net N$5: C201.1, IC1.20, R201.1
- new net N$6: C221.1, IC1.23, X1.P$3
- new net N$7: C231.1, IC1.22, X1.P$1
- new net N$8: C401.1, IC1.40
- new net N$9: IC1.30, L301.1
- new net P2_1: IC1.35, U$1.38
- new net P2_2: IC1.34, U$1.36
- new net RESET_N: R201.2, U$1.35
- net +3V3: now also L1.1, R32.1; no longer R1.2, U$3.VCC
- net GND: now also C101.2, C201.2, C21.2, C211.2, C221.2, C231.2, C241.2, C271.2, C272.2, C31.2, C311.2, C391.2, C4.2, C401.2, C41.2, C5.2, IC1.1, IC1.EXP, R301.1, U$4.GND, U1.P$2, U1.P$5, U1.P$6, USB1.4, USB1.5; no longer U$3.GND
Routing:
- net GND: track 91.8 -> 14.4 mm, vias 4 -> 0
- net RST: track 53.4 -> 0.00 mm
- net +3V3: track 51.9 -> 0.00 mm
- net DD: track 35.6 -> 0.00 mm
- net DC: track 34.2 -> 0.00 mm
- net E18-RX: track 28.4 -> 0.00 mm
- net E18-TX: track 27.9 -> 0.00 mm
- net N$7: track 0.00 -> 9.39 mm
- net N$6: track 0.00 -> 9.23 mm
- net N$15: track 0.00 -> 8.06 mm, vias 0 -> 2
- net +5V: track 38.0 -> 35.4 mm
