File: smart-home.matherboard.brd (EAGLE design)
At the start: 78 x 54 mm, 6 parts

Commit message: update schema
Parts:
- removed R1: 10kOm, rcl:R0603
- removed U$3: E18-MS1PA1IPX, e18-ms1pa1-ipx:E18-MS1PA1-IPX
- added C1: 100n, rcl:C0603K
- added J1: A2501WV-03P, jt:A2501WV-03P
- added J2: A2501WV-04P, jt:A2501WV-04P
- added R3, R4, R5: 10kOm, rcl:R0603
- added U1: CC2652P2-DUOWEISI, codm:CC2653P2-DUOWEISI
Connections:
- removed net CSN: U$3.P1.4
- removed net E18-RX: U$1.8, U$3.P0.2
- removed net E18-TX: U$1.10, U$3.P0.3
- removed net MISO: U$3.P1.7
- removed net MOSI: U$3.P1.6
- removed net RST: R1.1, U$1.35, U$3.RST
- removed net SCK: U$3.P1.5
- new net BSL_TRIGGER: R5.1, U$1.35, U1.DIO15
- new net CC_RX: U$1.8, U1.DIO12
- new net CC_TX: U$1.10, U1.DIO13
- new net DHT_PIN: J1.P2, R3.1, U$1.32
- new net I2C-CLOCK: J2.P3, U$1.5
- new net I2C-DATA: J2.P2, U$1.3
- new net JRES: R4.1, U$1.26, U1.RES
- new net JTCK: U$1.23, U1.TCKC
- new net JTDI: U$1.19, U1.DIO17
- new net JTDO: U$1.21, U1.DIO16
- new net JTMS: U$1.22, U1.TMSC
- net +3V3: now also C1.1, J1.P1, J2.P1, R3.2, R4.2, R5.2, U1.VCC; no longer R1.2, U$3.VCC
- net DC: no longer U$3.P2.2
- net DD: no longer U$3.P2.1
- net GND: now also C1.2, J1.P3, J2.P4, U1.GND, U1.GND@1; no longer U$3.GND
Routing:
- net +3V3: track 51.9 -> 128.8 mm, vias 0 -> 2
- net GND: track 91.8 -> 26.3 mm, vias 4 -> 2
- net JRES: track 0.00 -> 55.1 mm, vias 0 -> 1
- net RST: track 53.4 -> 0.00 mm
- net DHT_PIN: track 0.00 -> 51.2 mm
- net CC_RX: track 0.00 -> 37.4 mm, vias 0 -> 1
- net CC_TX: track 0.00 -> 36.9 mm, vias 0 -> 1
- net DD: track 35.6 -> 0.00 mm
- net DC: track 34.2 -> 0.00 mm
- net JTMS: track 0.00 -> 29.6 mm, vias 0 -> 1
- net E18-RX: track 28.4 -> 0.00 mm
- net E18-TX: track 27.9 -> 0.00 mm
- net JTCK: track 0.00 -> 26.0 mm, vias 0 -> 1
- net BSL_TRIGGER: track 0.00 -> 21.7 mm
- net I2C-DATA: track 0.00 -> 18.4 mm
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