File: smart-home.matherboard.sch (EAGLE design)
At the start: 5 parts

Commit message: update schema
Parts:
- removed R1: 10kOm, rcl:R-EU_R0603
- removed U$3: E18-MS1PA1IPX, e18-ms1pa1-ipx:E18-MS1PA1IPX
- added C1: 100n, rcl:C-EUC0603K
- added J1: A2501WV-03P, jt:A2501WV-03P
- added J2: A2501WV-04P, jt:A2501WV-04P
- added R3, R4, R5: 10kOm, rcl:R-EU_R0603
- added U1: CC2652P2-DUOWEISI, codm:CC2652P2-DUOWEISI
Connections:
- removed net CSN: U$3.P1.4
- removed net E18-RX: U$1.TXD0/GPIO14, U$3.P0.2
- removed net E18-TX: U$1.RXD0/GPIO15, U$3.P0.3
- removed net MISO: U$3.P1.7
- removed net MOSI: U$3.P1.6
- removed net RST: R1.1, U$1.GPIO19, U$3.RST
- removed net SCK: U$3.P1.5
- new net BSL_TRIGGER: R5.1, U$1.GPIO19, U1.DIO15
- new net CC_RX: U$1.TXD0/GPIO14, U1.DIO12
- new net CC_TX: U$1.RXD0/GPIO15, U1.DIO13
- new net DHT_PIN: J1.2, R3.1, U$1.GPIO12
- new net I2C-CLOCK: J2.3, U$1.GPIO3/SCL1
- new net I2C-DATA: J2.2, U$1.GPIO2/SDA1
- new net JRES: R4.1, U$1.!CE!/GPIO7, U1.RES
- new net JTCK: U$1.GPIO11/SCLK, U1.TCKC
- new net JTDI: U$1.GPIO10/MOSI, U1.DIO17
- new net JTDO: U$1.GPIO9/MISO, U1.DIO16
- new net JTMS: U$1.GEN/6GPIO25, U1.TMSC
- net +3V3: now also C1.1, J1.1, J2.1, R3.2, R4.2, R5.2, U1.VCC; no longer R1.2, U$3.VCC
- net DC: no longer U$3.P2.2
- net DD: no longer U$3.P2.1
- net GND: now also C1.2, J1.3, J2.4, U1.GND, U1.GND@1; no longer U$3.GND
Other:
- moved on the sheet: U$1
