File: hardware/smart-home.matherboard.sch (EAGLE design)
At the start: 10 parts, among them J1 A2501WV-03P, J2 A2501WV-04P, U1 CC2652P2-DUOWEISI

Commit message: Add buttons for reset and flash
Parts:
- added ZB-BSL, ZB-RST: SKRKAEE020, switch:SKRKAEE020
Connections:
- net BSL_TRIGGER: now also ZB-BSL.2
- net GND: now also ZB-BSL.1, ZB-RST.1
- net JRES: now also ZB-RST.2
Changed lines of the file:
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@@
 <layer number="56" name="wert" color="7" fill="1" visible="no" active="no"/>
 <layer number="57" name="tCAD" color="7" fill="1" visible="no" active="no"/>
+<layer number="58" name="bCAD" color="7" fill="1" visible="no" active="no"/>
 <layer number="59" name="tCarbon" color="7" fill="1" visible="no" active="no"/>
 <layer number="60" name="bCarbon" color="7" fill="1" visible="no" active="no"/>
+<layer number="61" name="stand" color="7" fill="1" visible="no" active="no"/>
 <layer number="88" name="SimResults" color="9" fill="1" visible="yes" active="yes"/>
 <layer number="89" name="SimProbes" color="9" fill="1" visible="yes" active="yes"/>
@@
 <layer number="154" name="FabDoc2" color="7" fill="1" visible="yes" active="yes"/>
 <layer number="155" name="FabDoc3" color="7" fill="1" visible="yes" active="yes"/>
+<layer number="160" name="O_Dim" color="7" fill="1" visible="no" active="yes"/>
+<layer number="166" name="AntennaArea" color="7" fill="1" visible="no" active="no"/>
+<layer number="168" name="4mmHeightArea" color="7" fill="1" visible="no" active="no"/>
 <layer number="191" name="mNets" color="7" fill="1" visible="yes" active="yes"/>
 <layer number="192" name="mBusses" color="7" fill="1" visible="yes" active="yes"/>
@@
 <part name="+3V6" library="supply1" library_urn="urn:adsk.eagle:library:371" deviceset="+3V3" device=""/>
 <part name="GND8" library="supply1" library_urn="urn:adsk.eagle:library:371" deviceset="GND" device=""/>
+<part name="ZB-RST" library="switch" deviceset="SKRKAEE020" device=""/>
+<part name="GND9" library="supply1" library_urn="urn:adsk.eagle:library:371" deviceset="GND" device=""/>
+<part name="ZB-BSL" library="switch" deviceset="SKRKAEE020" device=""/>
+<part name="GND10" library="supply1" library_urn="urn:adsk.eagle:library:371" deviceset="GND" device=""/>
 </parts>
 <sheets>
@@
 <instance part="GND8" gate="1" x="223.52" y="134.62" smashed="yes" grouprefs="I2C">
 <attribute name="VALUE" x="220.98" y="132.08" size="1.778" layer="96"/>
+</instance>
+<instance part="ZB-RST" gate="G$1" x="45.72" y="96.52" smashed="yes" grouprefs="ZIGBEE">
+<attribute name="NAME" x="39.37" y="92.075" size="1.778" layer="95" rot="R90"/>
+<attribute name="VALUE" x="49.53" y="86.995" size="1.778" layer="96" rot="R90"/>
+</instance>
+<instance part="GND9" gate="1" x="45.72" y="86.36" smashed="yes" grouprefs="ZIGBEE">
+<attribute name="VALUE" x="43.18" y="83.82" size="1.778" layer="96"/>
+</instance>
+<instance part="ZB-BSL" gate="G$1" x="152.4" y="88.9" smashed="yes" grouprefs="ZIGBEE">
+<attribute name="NAME" x="146.05" y="84.455" size="1.778" layer="95" rot="R90"/>
+<attribute name="VALUE" x="156.972" y="78.105" size="1.778" layer="96" rot="R90"/>
+</instance>
+<instance part="GND10" gate="1" x="152.4" y="78.74" smashed="yes" grouprefs="ZIGBEE">
+<attribute name="VALUE" x="149.86" y="76.2" size="1.778" layer="96"/>
 </instance>
 </instances>
@@
 <wire x1="223.52" y1="142.24" x2="223.52" y2="137.16" width="0.1524" layer="91" grouprefs="I2C"/>
 </segment>
+<segment>
+<pinref part="ZB-RST" gate="G$1" pin="1"/>
+<pinref part="GND9" gate="1" pin="GND"/>
+<wire x1="45.72" y1="91.44" x2="45.72" y2="88.9" width="0.1524" layer="91" grouprefs="ZIGBEE"/>
+</segment>
+<segment>
+<pinref part="GND10" gate="1" pin="GND"/>
+<pinref part="ZB-BSL" gate="G$1" pin="1"/>
+<wire x1="152.4" y1="81.28" x2="152.4" y2="83.82" width="0.1524" layer="91" grouprefs="ZIGBEE"/>
+</segment>
 </net>
 <net name="+5V" class="0">
@@
 <wire x1="45.72" y1="106.68" x2="45.72" y2="104.14" width="0.1524" layer="91" grouprefs="ZIGBEE"/>
 <junction x="45.72" y="104.14" grouprefs="ZIGBEE"/>
+<pinref part="ZB-RST" gate="G$1" pin="2"/>
+<wire x1="45.72" y1="104.14" x2="45.72" y2="101.6" width="0.1524" layer="91" grouprefs="ZIGBEE"/>
 </segment>
 <segment>
@@
 <wire x1="152.4" y1="99.06" x2="152.4" y2="96.52" width="0.1524" layer="91" grouprefs="ZIGBEE"/>
 <junction x="152.4" y="96.52" grouprefs="ZIGBEE"/>
-</segment>
-<segment>
+<pinref part="ZB-BSL" gate="G$1" pin="2"/>
+<wire x1="152.4" y1="93.98" x2="152.4" y2="96.52" width="0.1524" layer="91" grouprefs="ZIGBEE"/>
+</segment>
+<segment>
